File: Board/LED-Cube_v.brd (EAGLE design)
At the start: 150.4 x 120 mm, 119 parts, among them IC1 74HC595N, IC2 74HC595N, IC3 74HC595N, IC4 74HC595N, IC5 74HC595N, IC6 74HC595N, IC7 74HC595N, IC8 74HC595N, IC9 74HC595N, Q1 BC447, Q2 BC447, Q3 BC447, T1 TIP122, T2 TIP122, T3 TIP122, T4 TIP122, T5 TIP122, T6 TIP122, T7 TIP122, T8 TIP122

Commit message: last
Parts:
- moved U$1 99.8 mm to (143.0, 64.0), turned to 270 degrees
- moved Q1 6.08 mm to (42.8, 40.4)
- moved Q3 3.00 mm to (50.8, 46.5)
Routing:
- net GND: track 828.9 -> 823.5 mm
- net N$5: track 3.30 -> 8.54 mm
- net DATA: track 66.0 -> 70.7 mm
- net N$2: track 10.4 -> 11.7 mm
- net VCC: track 602.5 -> 603.7 mm
Other:
- outline, holes or cut-outs redrawn
- board text added: "5V"
- board text added: "D"
- board text added: "L"
- board text added: "S"
- board text added: "USB"
