File: Board/LED-Cube_v2.sch (EAGLE design)
At the start: 113 parts, among them IC1 74HC595N, IC2 74HC595N, IC3 74HC595N, IC4 74HC595N, IC5 74HC595N, IC6 74HC595N, IC7 74HC595N, IC8 74HC595N, IC9 74HC595N, J1 DCJ0202, Q1 BC447, Q2 BC447, Q3 BC447, T1 TIP122, T2 TIP122, T3 TIP122, T4 TIP122, T5 TIP122, T6 TIP122, T7 TIP122, T8 TIP122

Commit message: last
Parts:
- removed J1: DCJ0202, con-jack:DCJ0202
- added J2: (no value), 5mm_more_width:DCJ0303
- added PAD1, PAD2, PAD3, PAD4: (no value), wirepad:3,81/1,4
Connections:
- net GND: now also J2.3; no longer J1.3
- net VCC: now also J2.1; no longer J1.1
Changed lines of the file:
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@@
 <part name="R50" library="rcl" deviceset="R-EU_" device="0207/10"/>
 <part name="R51" library="rcl" deviceset="R-EU_" device="0207/10"/>
-<part name="J1" library="con-jack" deviceset="DCJ0202" device=""/>
 <part name="IC8" library="74xx-eu" deviceset="74*595" device="N" technology="HC"/>
 <part name="JP8" library="pinhead" deviceset="PINHD-1X8" device=""/>
@@
 <part name="R77" library="rcl" deviceset="R-EU_" device="0207/10"/>
 <part name="R78" library="rcl" deviceset="R-EU_" device="0207/10"/>
-<part name="U$2" library="PI_PICO" deviceset="PI_PICO" device=""/>
 <part name="R79" library="rcl" deviceset="R-EU_" device="0207/10"/>
 <part name="R80" library="rcl" deviceset="R-EU_" device="0207/10"/>
 <part name="SV1" library="con-lstb" library_urn="urn:adsk.eagle:library:162" deviceset="MA03-1" device="" package3d_urn="urn:adsk.eagle:package:8339/1"/>
 <part name="SV2" library="con-lstb" library_urn="urn:adsk.eagle:library:162" deviceset="MA05-1" device="" package3d_urn="urn:adsk.eagle:package:8332/1"/>
+<part name="U$2" library="PI_PICO" deviceset="PI_PICO" device=""/>
+<part name="J2" library="5mm_more_width" deviceset="DCJ0303" device="" package3d_urn="urn:adsk.eagle:package:7493/1"/>
+<part name="PAD1" library="wirepad" library_urn="urn:adsk.eagle:library:412" deviceset="3,81/1,4" device="" package3d_urn="urn:adsk.eagle:package:30835/1"/>
+<part name="PAD2" library="wirepad" library_urn="urn:adsk.eagle:library:412" deviceset="3,81/1,4" device="" package3d_urn="urn:adsk.eagle:package:30835/1"/>
+<part name="PAD3" library="wirepad" library_urn="urn:adsk.eagle:library:412" deviceset="3,81/1,4" device="" package3d_urn="urn:adsk.eagle:package:30835/1"/>
+<part name="PAD4" library="wirepad" library_urn="urn:adsk.eagle:library:412" deviceset="3,81/1,4" device="" package3d_urn="urn:adsk.eagle:package:30835/1"/>
 </parts>
 <sheets>
@@
 <attribute name="VALUE" x="433.07" y="55.118" size="1.778" layer="96"/>
 </instance>
-<instance part="J1" gate="G$1" x="60.96" y="71.12" smashed="yes">
-<attribute name="NAME" x="58.42" y="74.93" size="1.778" layer="95"/>
-<attribute name="VALUE" x="58.42" y="64.77" size="1.778" layer="96"/>
-</instance>
 <instance part="IC8" gate="A" x="477.52" y="66.04" smashed="yes">
 <attribute name="NAME" x="469.9" y="79.375" size="1.778" layer="95"/>
@@
 <attribute name="VALUE" x="82.55" y="-28.702" size="1.778" layer="96"/>
 </instance>
-<instance part="U$2" gate="G$1" x="33.02" y="33.02" smashed="yes"/>
 <instance part="R79" gate="G$1" x="22.86" y="91.44" smashed="yes" rot="R180">
 <attribute name="NAME" x="26.67" y="89.9414" size="1.778" layer="95" rot="R180"/>
@@
 <attribute name="VALUE" x="67.31" y="48.26" size="1.778" layer="96" rot="R180"/>
 <attribute name="NAME" x="67.31" y="29.718" size="1.778" layer="95" rot="R180"/>
+</instance>
+<instance part="U$2" gate="G$1" x="33.02" y="33.02" smashed="yes"/>
+<instance part="J2" gate="G$1" x="60.96" y="71.12" smashed="yes">
+<attribute name="NAME" x="58.42" y="74.93" size="1.778" layer="95"/>
+<attribute name="VALUE" x="58.42" y="64.77" size="1.778" layer="96"/>
+</instance>
+<instance part="PAD1" gate="1" x="127" y="-2.54" smashed="yes">
+<attribute name="NAME" x="125.857" y="-0.6858" size="1.778" layer="95"/>
+<attribute name="VALUE" x="125.857" y="-5.842" size="1.778" layer="96"/>
+</instance>
+<instance part="PAD2" gate="1" x="137.16" y="-5.08" smashed="yes">
+<attribute name="NAME" x="136.017" y="-3.2258" size="1.778" layer="95"/>
+<attribute name="VALUE" x="136.017" y="-8.382" size="1.778" layer="96"/>
+</instance>
+<instance part="PAD3" gate="1" x="147.32" y="-5.08" smashed="yes">
+<attribute name="NAME" x="146.177" y="-3.2258" size="1.778" layer="95"/>
+<attribute name="VALUE" x="146.177" y="-8.382" size="1.778" layer="96"/>
+</instance>
+<instance part="PAD4" gate="1" x="157.48" y="-5.08" smashed="yes">
+<attribute name="NAME" x="156.337" y="-3.2258" size="1.778" layer="95"/>
+<attribute name="VALUE" x="156.337" y="-8.382" size="1.778" layer="96"/>
 </instance>
 </instances>
@@
 <wire x1="55.88" y1="-30.48" x2="60.96" y2="-30.48" width="0.1524" layer="91"/>
 <wire x1="55.88" y1="-30.48" x2="55.88" y2="10.16" width="0.1524" layer="91"/>
+<wire x1="55.88" y1="10.16" x2="48.26" y2="10.16" width="0.1524" layer="91"/>
 <pinref part="U$2" gate="G$1" pin="GP17"/>
-<wire x1="55.88" y1="10.16" x2="48.26" y2="10.16" width="0.1524" layer="91"/>
 </segment>
 </net>
@@
 <junction x="86.36" y="68.58"/>
 <wire x1="86.36" y1="68.58" x2="86.36" y2="63.5" width="0.1524" layer="91"/>
-<pinref part="J1" gate="G$1" pin="1"/>
 <wire x1="68.58" y1="73.66" x2="73.66" y2="73.66" width="0.1524" layer="91"/>
 <wire x1="73.66" y1="73.66" x2="73.66" y2="63.5" width="0.1524" layer="91"/>
@@
 <wire x1="93.98" y1="27.94" x2="93.98" y2="53.34" width="0.1524" layer="91"/>
 <junction x="93.98" y="27.94"/>
-<pinref part="U$2" gate="G$1" pin="VSYS"/>
 <wire x1="7.62" y1="96.52" x2="53.34" y2="96.52" width="0.1524" layer="91"/>
 <wire x1="53.34" y1="96.52" x2="53.34" y2="53.34" width="0.1524" layer="91"/>
@@
 <wire x1="58.42" y1="33.02" x2="58.42" y2="27.94" width="0.1524" layer="91"/>
 <wire x1="58.42" y1="27.94" x2="93.98" y2="27.94" width="0.1524" layer="91"/>
+<pinref part="U$2" gate="G$1" pin="VSYS"/>
+<pinref part="J2" gate="G$1" pin="1"/>
 </segment>
 </net>
@@
 <junction x="345.44" y="38.1"/>
 <junction x="81.28" y="50.8"/>
-<pinref part="J1" gate="G$1" pin="3"/>
 <wire x1="81.28" y1="68.58" x2="81.28" y2="50.8" width="0.1524" layer="91"/>
 <wire x1="68.58" y1="68.58" x2="81.28" y2="68.58" width="0.1524" layer="91"/>
@@
 <wire x1="78.74" y1="-17.78" x2="96.52" y2="-17.78" width="0.1524" layer="91"/>
 <junction x="96.52" y="-17.78"/>
-<pinref part="U$2" gate="G$1" pin="GND8"/>
 <wire x1="586.74" y1="38.1" x2="665.48" y2="38.1" width="0.1524" layer="91"/>
 <wire x1="665.48" y1="38.1" x2="665.48" y2="33.02" width="0.1524" layer="91"/>
@@
 <wire x1="58.42" y1="43.18" x2="58.42" y2="50.8" width="0.1524" layer="91"/>
 <junction x="58.42" y="50.8"/>
+<pinref part="U$2" gate="G$1" pin="GND8"/>
+<pinref part="J2" gate="G$1" pin="3"/>
 </segment>
 </net>
@@
 <wire x1="53.34" y1="7.62" x2="53.34" y2="-12.7" width="0.1524" layer="91"/>
 <wire x1="53.34" y1="-12.7" x2="60.96" y2="-12.7" width="0.1524" layer="91"/>
+<wire x1="53.34" y1="7.62" x2="48.26" y2="7.62" width="0.1524" layer="91"/>
 <pinref part="U$2" gate="G$1" pin="GP16"/>
-<wire x1="53.34" y1="7.62" x2="48.26" y2="7.62" width="0.1524" layer="91"/>
 </segment>
 </net>
@@
 <wire x1="7.62" y1="93.98" x2="15.24" y2="93.98" width="0.1524" layer="91"/>
 <pinref part="SV1" gate="G$1" pin="2"/>
-<pinref part="U$2" gate="G$1" pin="GP0"/>
 <wire x1="15.24" y1="93.98" x2="17.78" y2="93.98" width="0.1524" layer="91"/>
 <wire x1="17.78" y1="55.88" x2="15.24" y2="55.88" width="0.1524" layer="91"/>
 <wire x1="15.24" y1="55.88" x2="15.24" y2="93.98" width="0.1524" layer="91"/>
 <junction x="15.24" y="93.98"/>
+<pinref part="U$2" gate="G$1" pin="GP0"/>
 </segment>
 </net>
 <net name="N$43" class="0">
 <segment>
-<pinref part="U$2" gate="G$1" pin="GP1"/>
 <wire x1="17.78" y1="53.34" x2="12.7" y2="53.34" width="0.1524" layer="91"/>
 <pinref part="R79" gate="G$1" pin="2"/>
@@
 <wire x1="12.7" y1="53.34" x2="12.7" y2="91.44" width="0.1524" layer="91"/>
 <junction x="12.7" y="91.44"/>
+<pinref part="U$2" gate="G$1" pin="GP1"/>
 </segment>
 </net>
 <net name="N$3" class="0">
 <segment>
-<pinref part="U$2" gate="G$1" pin="GP26"/>
 <wire x1="48.26" y1="33.02" x2="55.88" y2="33.02" width="0.1524" layer="91"/>
 <wire x1="55.88" y1="33.02" x2="55.88" y2="35.56" width="0.1524" layer="91"/>
 <pinref part="SV2" gate="G$1" pin="4"/>
 <wire x1="55.88" y1="35.56" x2="58.42" y2="35.56" width="0.1524" layer="91"/>
+<pinref part="U$2" gate="G$1" pin="GP26"/>
 </segment>
 </net>
 <net name="N$118" class="0">
 <segment>
-<pinref part="U$2" gate="G$1" pin="GP27"/>
 <wire x1="48.26" y1="35.56" x2="53.34" y2="35.56" width="0.1524" layer="91"/>
 <wire x1="53.34" y1="35.56" x2="53.34" y2="38.1" width="0.1524" layer="91"/>
 <pinref part="SV2" gate="G$1" pin="3"/>
 <wire x1="53.34" y1="38.1" x2="58.42" y2="38.1" width="0.1524" layer="91"/>
+<pinref part="U$2" gate="G$1" pin="GP27"/>
 </segment>
 </net>
 <net name="N$153" class="0">
 <segment>
-<pinref part="U$2" gate="G$1" pin="GP28"/>
 <pinref part="SV2" gate="G$1" pin="2"/>
 <wire x1="48.26" y1="40.64" x2="58.42" y2="40.64" width="0.1524" layer="91"/>
-</segment>
-</net>
+<pinref part="U$2" gate="G$1" pin="GP28"/>
+</segment>
+</net>
