File: Board/Pin-Zusammenfassung.brd (EAGLE design)
At the start: 109.4 x 11.9 mm, 9 parts

Commit message: last
Parts:
- added U$1: (no value), HTL-Logo:LOGOBOT_8
- moved JP1 0.84 mm to (67.5, 9.29)
Routing:
- net N$7: track 35.3 -> 34.3 mm
- net N$3: track 22.9 -> 22.0 mm
- net N$5: track 10.9 -> 10.0 mm
- net N$4: track 10.9 -> 10.0 mm
- net N$2: track 35.1 -> 34.4 mm
Other:
- board size 109.4 x 11.9 mm -> 109.4 x 11.1 mm
- board text added: "BS 3AHET"
- board text added: "Pin-Zusammenfassung"
Changed lines of the file:
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@@
 <setting verticaltext="up"/>
 </settings>
-<grid distance="590.551181" unitdist="mil" unit="mil" style="dots" multiple="1" display="yes" altdistance="0.01" altunitdist="mm" altunit="mm"/>
+<grid distance="15" unitdist="mm" unit="mm" style="dots" multiple="1" display="yes" altdistance="0.01" altunitdist="mm" altunit="mm"/>
 <layers>
 <layer number="1" name="Top" color="4" fill="1" visible="yes" active="yes"/>
@@
 <board>
 <plain>
-<wire x1="12.79" y1="5.38" x2="122.22" y2="5.38" width="0.4064" layer="20"/>
-<wire x1="122.22" y1="5.38" x2="122.22" y2="17.27" width="0.4064" layer="20"/>
+<wire x1="12.79" y1="6.19" x2="122.21" y2="6.14" width="0.4064" layer="20"/>
+<wire x1="122.21" y1="6.14" x2="122.22" y2="17.27" width="0.4064" layer="20"/>
 <wire x1="122.22" y1="17.27" x2="12.79" y2="17.22" width="0.4064" layer="20"/>
-<wire x1="12.79" y1="17.22" x2="12.79" y2="5.38" width="0.4064" layer="20"/>
+<wire x1="12.79" y1="17.22" x2="12.79" y2="6.19" width="0.4064" layer="20"/>
+<text x="46.75" y="7.64" size="1.778" layer="16" font="vector" ratio="16" rot="MR0">BS 3AHET</text>
+<text x="112.74" y="7.57" size="1.778" layer="16" font="vector" ratio="16" rot="MR0">Pin-Zusammenfassung</text>
 </plain>
 <attributes>
@@
 </autorouter>
 <elements>
-<element name="JP1" library="pinhead" library_urn="urn:adsk.eagle:library:325" package="1X08" package3d_urn="urn:adsk.eagle:package:22409/2" value="" x="67.49" y="8.45" smashed="yes">
-<attribute name="NAME" x="57.2538" y="10.2788" size="1.27" layer="25" ratio="10"/>
-<attribute name="POPULARITY" value="67" x="91.62" y="5.91" size="1.778" layer="27" display="off"/>
-<attribute name="VALUE" x="57.33" y="5.275" size="1.27" layer="27"/>
+<element name="JP1" library="pinhead" library_urn="urn:adsk.eagle:library:325" package="1X08" package3d_urn="urn:adsk.eagle:package:22409/2" value="" x="67.49" y="9.29" smashed="yes">
+<attribute name="NAME" x="57.2538" y="11.1188" size="1.27" layer="25" ratio="10"/>
+<attribute name="POPULARITY" value="67" x="91.62" y="6.75" size="1.778" layer="27" display="off"/>
+<attribute name="VALUE" x="57.33" y="6.115" size="1.27" layer="27"/>
 </element>
 <element name="JP2" library="pinhead" library_urn="urn:adsk.eagle:library:325" package="1X01" package3d_urn="urn:adsk.eagle:package:22485/2" value="" x="120.01" y="15" smashed="yes">
@@
 <attribute name="VALUE" x="13.73" y="11.825" size="1.27" layer="27"/>
 </element>
+<element name="U$1" library="HTL-Logo" package="LOGOBOT_8" value="" x="27.39" y="8.11" smashed="yes"/>
 </elements>
 <signals>
@@
 <contactref element="JP1" pad="8"/>
 <contactref element="JP2" pad="1"/>
-<wire x1="115.36" y1="10.35" x2="78.78" y2="10.35" width="0.8128" layer="16"/>
-<wire x1="78.78" y1="10.35" x2="76.88" y2="8.45" width="0.8128" layer="16"/>
-<wire x1="76.38" y1="8.45" x2="76.88" y2="8.45" width="0.8128" layer="16"/>
-<wire x1="115.36" y1="10.35" x2="120.01" y2="15" width="0.8128" layer="16"/>
+<wire x1="115.76" y1="10.75" x2="78.42" y2="10.75" width="0.8128" layer="16"/>
+<wire x1="78.42" y1="10.75" x2="76.96" y2="9.29" width="0.8128" layer="16"/>
+<wire x1="76.38" y1="9.29" x2="76.96" y2="9.29" width="0.8128" layer="16"/>
+<wire x1="115.76" y1="10.75" x2="120.01" y2="15" width="0.8128" layer="16"/>
 </signal>
 <signal name="N$2">
 <contactref element="JP1" pad="7"/>
 <contactref element="JP3" pad="1"/>
-<wire x1="73.84" y1="8.45" x2="74" y2="8.61" width="0.508" layer="16"/>
-<wire x1="74" y1="8.61" x2="74" y2="10.67" width="0.8128" layer="16"/>
-<wire x1="74" y1="10.67" x2="74.93" y2="11.6" width="0.8128" layer="16"/>
-<wire x1="74.93" y1="11.6" x2="101.61" y2="11.6" width="0.8128" layer="16"/>
-<wire x1="101.61" y1="11.6" x2="105.01" y2="15" width="0.8128" layer="16"/>
+<wire x1="73.84" y1="9.29" x2="73.89" y2="9.34" width="0.508" layer="16"/>
+<wire x1="73.89" y1="9.34" x2="73.89" y2="10.82" width="0.8128" layer="16"/>
+<wire x1="73.89" y1="10.82" x2="75.07" y2="12" width="0.8128" layer="16"/>
+<wire x1="75.07" y1="12" x2="102.01" y2="12" width="0.8128" layer="16"/>
+<wire x1="102.01" y1="12" x2="105.01" y2="15" width="0.8128" layer="16"/>
 </signal>
 <signal name="N$3">
 <contactref element="JP1" pad="6"/>
 <contactref element="JP4" pad="1"/>
-<wire x1="89.99" y1="13.99" x2="89" y2="13" width="0.8128" layer="16"/>
-<wire x1="89" y1="13" x2="74.19" y2="13" width="0.8128" layer="16"/>
-<wire x1="71.3" y1="10.11" x2="71.3" y2="8.45" width="0.8128" layer="16"/>
-<wire x1="74.19" y1="13" x2="71.3" y2="10.11" width="0.8128" layer="16"/>
-<wire x1="89.99" y1="14.98" x2="89.99" y2="13.99" width="0.8128" layer="16"/>
+<wire x1="89.99" y1="14.98" x2="88.23" y2="13.22" width="0.8128" layer="16"/>
+<wire x1="88.23" y1="13.22" x2="73.52" y2="13.22" width="0.8128" layer="16"/>
+<wire x1="71.3" y1="11" x2="71.3" y2="9.29" width="0.8128" layer="16"/>
+<wire x1="73.52" y1="13.22" x2="71.3" y2="11" width="0.8128" layer="16"/>
 </signal>
 <signal name="N$4">
@@
 <contactref element="JP5" pad="1"/>
 <wire x1="74.99" y1="14.99" x2="71.99" y2="14.99" width="0.8128" layer="16"/>
-<wire x1="68.76" y1="11.76" x2="68.76" y2="8.45" width="0.8128" layer="16"/>
+<wire x1="68.76" y1="11.76" x2="68.76" y2="9.29" width="0.8128" layer="16"/>
 <wire x1="71.99" y1="14.99" x2="68.76" y2="11.76" width="0.8128" layer="16"/>
 </signal>
@@
 <contactref element="JP6" pad="1"/>
 <wire x1="60" y1="14.98" x2="63.02" y2="14.98" width="0.8128" layer="16"/>
-<wire x1="66.22" y1="11.78" x2="66.22" y2="8.45" width="0.8128" layer="16"/>
+<wire x1="66.22" y1="11.78" x2="66.22" y2="9.29" width="0.8128" layer="16"/>
 <wire x1="63.02" y1="14.98" x2="66.22" y2="11.78" width="0.8128" layer="16"/>
 </signal>
@@
 <contactref element="JP1" pad="3"/>
 <contactref element="JP7" pad="1"/>
-<wire x1="60.96" y1="12.84" x2="47.18" y2="12.84" width="0.8128" layer="16"/>
-<wire x1="45.01" y1="15.01" x2="47.18" y2="12.84" width="0.8128" layer="16"/>
-<wire x1="63.68" y1="8.45" x2="63.68" y2="10.12" width="0.8128" layer="16"/>
-<wire x1="63.68" y1="10.12" x2="60.96" y2="12.84" width="0.8128" layer="16"/>
+<wire x1="61.82" y1="13.25" x2="46.77" y2="13.25" width="0.8128" layer="16"/>
+<wire x1="45.01" y1="15.01" x2="46.77" y2="13.25" width="0.8128" layer="16"/>
+<wire x1="63.68" y1="9.29" x2="63.68" y2="11.39" width="0.8128" layer="16"/>
+<wire x1="63.68" y1="11.39" x2="61.82" y2="13.25" width="0.8128" layer="16"/>
 </signal>
 <signal name="N$7">
 <contactref element="JP1" pad="2"/>
 <contactref element="JP8" pad="1"/>
-<wire x1="30" y1="15" x2="33.5" y2="11.5" width="0.8128" layer="16"/>
-<wire x1="61.14" y1="10.85" x2="61.14" y2="8.45" width="0.8128" layer="16"/>
-<wire x1="61.14" y1="10.85" x2="60.49" y2="11.5" width="0.8128" layer="16"/>
-<wire x1="33.5" y1="11.5" x2="60.49" y2="11.5" width="0.8128" layer="16"/>
+<wire x1="30" y1="15" x2="32.99" y2="12.01" width="0.8128" layer="16"/>
+<wire x1="61.14" y1="10.6" x2="61.14" y2="9.29" width="0.8128" layer="16"/>
+<wire x1="61.14" y1="10.6" x2="59.73" y2="12.01" width="0.8128" layer="16"/>
+<wire x1="32.99" y1="12.01" x2="59.73" y2="12.01" width="0.8128" layer="16"/>
 </signal>
 <signal name="N$8">
 <contactref element="JP1" pad="1"/>
 <contactref element="JP9" pad="1"/>
-<wire x1="15" y1="15" x2="15" y2="15.06" width="0.508" layer="16"/>
-<wire x1="15" y1="15" x2="19.75" y2="10.25" width="0.8128" layer="16"/>
-<wire x1="56.77" y1="10.25" x2="19.75" y2="10.25" width="0.8128" layer="16"/>
-<wire x1="58.57" y1="8.45" x2="58.6" y2="8.45" width="0.8128" layer="16"/>
-<wire x1="58.57" y1="8.45" x2="56.77" y2="10.25" width="0.8128" layer="16"/>
+<wire x1="56.84" y1="10.77" x2="19.23" y2="10.77" width="0.8128" layer="16"/>
+<wire x1="58.6" y1="9.29" x2="58.32" y2="9.29" width="0.8128" layer="16"/>
+<wire x1="58.32" y1="9.29" x2="56.84" y2="10.77" width="0.8128" layer="16"/>
+<wire x1="19.23" y1="10.77" x2="15" y2="15" width="0.8128" layer="16"/>
 </signal>
 <signal name="GND">
 <polygon width="0.4064" layer="16" isolate="0.8128">
 <vertex x="12.8" y="17.19"/>
-<vertex x="122.22" y="17.19"/>
-<vertex x="122.22" y="5.41"/>
-<vertex x="12.8" y="5.41"/>
+<vertex x="122.16" y="17.19"/>
+<vertex x="122.16" y="6.24"/>
+<vertex x="12.8" y="6.24"/>
 </polygon>
 </signal>
