File: Board/smalltest.sch (EAGLE design)
At the start: 113 parts, among them IC1 74HC595N, IC2 74HC595N, IC3 74HC595N, IC4 74HC595N, IC5 74HC595N, IC6 74HC595N, IC7 74HC595N, IC8 74HC595N, IC9 74HC595N, J1 DCJ0202, Q1 BC447, Q2 BC447, Q3 BC447, T1 TIP122, T2 TIP122, T3 TIP122, T4 TIP122, T5 TIP122, T6 TIP122, T7 TIP122, T8 TIP122

Commit message: new board
Parts:
- removed IC1, IC2, IC3, IC4, IC5, IC6, IC7, IC8, IC9: 74HC595N, 74xx-eu:74HC595N
- removed JP2, JP3, JP4, JP5, JP6, JP7, JP8, JP9: (no value), pinhead:PINHD-1X8
- removed R10, R11, R12, R13, R14, R15, R16, R17, R18, R19, R20, R21, R22, R23, R24, R25, R26, R27, R28, R29, R30, R31, R32, R33, R34, R35, R36, R37, R38, R39, R4, R40, R41, R42, R43, R44, R45, R46, R47, R48, R49, R5, R50, R51, R52, R53, R54, R55, R56, R57, R58, R59, R6, R60, R61, R62, R63, R64, R65, R66, R67, R68, R69, R7, R70, R71, R72, R73, R74, R75, R8, R9: (no value), rcl:R-EU_0207/10
- removed SV2: (no value), con-lstb:MA05-1
- removed T1, T2, T3, T4, T5, T6, T7, T8: TIP122, transistor:TIP122
- JP1: device pinhead:PINHD-1X8 -> pinhead:PINHD-1X5
Connections:
- removed net N$10: IC1A.QG, R10.1
- removed net N$100: IC7A.QF, R57.1
- removed net N$101: IC6A.QB, R45.1
- removed net N$102: IC6A.QC, R46.1
- removed net N$103: IC6A.QD, R47.1
- removed net N$104: IC6A.QE, R48.1
- removed net N$105: IC6A.QA, R44.1
- removed net N$106: IC6A.QF, R49.1
- removed net N$107: IC6A.QG, R50.1
- removed net N$108: IC6A.QH, R51.1
- removed net N$109: JP6.1, R44.2
- removed net N$11: IC1A.QH, R11.1
- removed net N$110: JP6.2, R45.2
- removed net N$111: JP6.3, R46.2
- removed net N$112: JP6.4, R47.2
- removed net N$113: JP6.5, R48.2
- removed net N$114: JP6.6, R49.2
- removed net N$115: JP6.7, R50.2
- removed net N$116: JP6.8, R51.2
- removed net N$117: IC7A.QG, R58.1
- removed net N$118: SV2.3, U$2.GP27
- removed net N$119: IC7A.QH, R59.1
- removed net N$12: JP1.1, R4.2
- removed net N$120: R52.2, T7.B
- removed net N$121: R53.2, T1.B
- removed net N$122: R54.2, T2.B
- removed net N$123: R55.2, T3.B
- removed net N$124: R56.2, T4.B
- removed net N$125: R57.2, T5.B
- removed net N$126: R58.2, T6.B
- removed net N$127: R59.2, T8.B
- removed net N$128: JP7.1, T7.C
- removed net N$129: JP7.2, T1.C
- removed net N$13: JP1.2, R5.2
- removed net N$130: JP7.3, T2.C
- removed net N$131: JP7.4, T3.C
- removed net N$132: JP7.5, T4.C
- removed net N$133: JP7.6, T5.C
- removed net N$134: JP7.7, T6.C
- removed net N$135: JP7.8, T8.C
- removed net N$136: IC6A.QH*, IC8A.SER
- removed net N$137: IC8A.QB, R61.1
- removed net N$138: IC8A.QC, R62.1
- removed net N$139: IC8A.QD, R63.1
- removed net N$14: IC1A.QB, R5.1
- removed net N$140: IC8A.QE, R64.1
- removed net N$141: IC8A.QA, R60.1
- removed net N$142: IC8A.QF, R65.1
- removed net N$143: IC8A.QG, R66.1
- removed net N$144: IC8A.QH, R67.1
- removed net N$145: JP8.1, R60.2
- removed net N$146: JP8.2, R61.2
- removed net N$147: JP8.3, R62.2
- removed net N$148: JP8.4, R63.2
- removed net N$149: JP8.5, R64.2
- removed net N$15: IC1A.QC, R6.1
- removed net N$150: JP8.6, R65.2
- removed net N$151: JP8.7, R66.2
- removed net N$152: JP8.8, R67.2
- removed net N$153: SV2.2, U$2.GP28
- removed net N$154: IC8A.QH*, IC9A.SER
- removed net N$155: IC9A.QB, R69.1
- removed net N$156: IC9A.QC, R70.1
- removed net N$157: IC9A.QD, R71.1
- removed net N$158: IC9A.QE, R72.1
- removed net N$159: IC9A.QA, R68.1
- removed net N$16: IC1A.QD, R7.1
- removed net N$160: IC9A.QF, R73.1
- removed net N$161: IC9A.QG, R74.1
- removed net N$162: IC9A.QH, R75.1
- removed net N$163: JP9.1, R68.2
- removed net N$164: JP9.2, R69.2
- removed net N$165: JP9.3, R70.2
- removed net N$166: JP9.4, R71.2
- removed net N$167: JP9.5, R72.2
- removed net N$168: JP9.6, R73.2
- removed net N$169: JP9.7, R74.2
- removed net N$17: IC1A.QE, R8.1
- removed net N$170: JP9.8, R75.2
- removed net N$173: IC7A.SER, IC9A.QH*
- removed net N$18: JP1.3, R6.2
- removed net N$19: JP1.4, R7.2
- removed net N$20: JP1.5, R8.2
- removed net N$21: JP1.6, R9.2
- removed net N$22: JP1.7, R10.2
- removed net N$23: JP1.8, R11.2
- removed net N$24: IC2A.QB, R13.1
- removed net N$25: IC2A.QC, R14.1
- removed net N$26: IC2A.QD, R15.1
- removed net N$27: IC2A.QE, R16.1
- removed net N$28: IC1A.QH*, IC2A.SER
- removed net N$29: IC2A.QA, R12.1
- removed net N$3: SV2.4, U$2.GP26
- removed net N$30: IC2A.QF, R17.1
- removed net N$31: IC2A.QG, R18.1
- removed net N$32: IC2A.QH, R19.1
- removed net N$33: JP2.1, R12.2
- removed net N$34: JP2.2, R13.2
- removed net N$35: JP2.3, R14.2
- removed net N$36: JP2.4, R15.2
- removed net N$37: JP2.5, R16.2
- removed net N$38: JP2.6, R17.2
- removed net N$39: JP2.7, R18.2
- removed net N$40: JP2.8, R19.2
- removed net N$42: IC2A.QH*, IC3A.SER
- removed net N$44: IC3A.QB, R21.1
- removed net N$45: IC3A.QC, R22.1
- removed net N$46: IC3A.QD, R23.1
- removed net N$47: IC3A.QE, R24.1
- removed net N$48: IC3A.QA, R20.1
- removed net N$49: IC3A.QF, R25.1
- removed net N$50: IC3A.QG, R26.1
- removed net N$51: IC3A.QH, R27.1
- removed net N$52: JP3.1, R20.2
- removed net N$53: JP3.2, R21.2
- removed net N$54: JP3.3, R22.2
- removed net N$55: JP3.4, R23.2
- removed net N$56: JP3.5, R24.2
- removed net N$57: JP3.6, R25.2
- removed net N$58: JP3.7, R26.2
- removed net N$59: JP3.8, R27.2
- removed net N$60: IC7A.QA, R52.1
- removed net N$61: IC3A.QH*, IC4A.SER
- removed net N$62: IC7A.QB, R53.1
- removed net N$63: IC4A.QB, R29.1
- removed net N$64: IC4A.QC, R30.1
- removed net N$65: IC4A.QD, R31.1
- removed net N$66: IC4A.QE, R32.1
- removed net N$67: IC4A.QA, R28.1
- removed net N$68: IC4A.QF, R33.1
- removed net N$69: IC4A.QG, R34.1
- removed net N$70: IC4A.QH, R35.1
- removed net N$71: JP4.1, R28.2
- removed net N$72: JP4.2, R29.2
- removed net N$73: JP4.3, R30.2
- removed net N$74: JP4.4, R31.2
- removed net N$75: JP4.5, R32.2
- removed net N$76: JP4.6, R33.2
- removed net N$77: JP4.7, R34.2
- removed net N$78: JP4.8, R35.2
- removed net N$79: IC7A.QC, R54.1
- removed net N$8: IC1A.QA, R4.1
- removed net N$80: IC4A.QH*, IC5A.SER
- removed net N$81: IC7A.QD, R55.1
- removed net N$82: IC5A.QB, R37.1
- removed net N$83: IC5A.QC, R38.1
- removed net N$84: IC5A.QD, R39.1
- removed net N$85: IC5A.QE, R40.1
- removed net N$86: IC5A.QA, R36.1
- removed net N$87: IC5A.QF, R41.1
- removed net N$88: IC5A.QG, R42.1
- removed net N$89: IC5A.QH, R43.1
- removed net N$9: IC1A.QF, R9.1
- removed net N$90: JP5.1, R36.2
- removed net N$91: JP5.2, R37.2
- removed net N$92: JP5.3, R38.2
- removed net N$93: JP5.4, R39.2
- removed net N$94: JP5.5, R40.2
- removed net N$95: JP5.6, R41.2
- removed net N$96: JP5.7, R42.2
- removed net N$97: JP5.8, R43.2
- removed net N$98: IC7A.QE, R56.1
- removed net N$99: IC5A.QH*, IC6A.SER
- net DATA: now also JP1.2; no longer IC1A.SER
- net GND: now also JP1.5; no longer IC1A.G, IC2A.G, IC3A.G, IC4A.G, IC5A.G, IC6A.G, IC7A.G, IC8A.G, IC9A.G, SV2.1, T1.E, T2.E, T3.E, T4.E, T5.E, T6.E, T7.E, T8.E
- net SHIFT: now also JP1.3; no longer IC1A.SCK, IC2A.SCK, IC3A.SCK, IC4A.SCK, IC5A.SCK, IC6A.SCK, IC7A.SCK, IC8A.SCK, IC9A.SCK
- net STORE: now also JP1.4; no longer IC1A.RCK, IC2A.RCK, IC3A.RCK, IC4A.RCK, IC5A.RCK, IC6A.RCK, IC7A.RCK, IC8A.RCK, IC9A.RCK
- net VCC: now also JP1.1; no longer IC1A.SCL, IC2A.SCL, IC3A.SCL, IC4A.SCL, IC5A.SCL, IC6A.SCL, IC7A.SCL, IC8A.SCL, IC9A.SCL, SV2.5
Other:
- note removed: "G"
- moved on the sheet: J1, Q1, Q2, Q3, R1, R2, R3, R76, R77, R78, R79, R80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
